File: Electrical/Drone.brd (EAGLE design)
At the start: 85 x 81.5 mm, 76 parts, among them IC1 EFM8BB21F16G-C-QFN20R, IC2 FD6288Q, IC3 LDL212PV33R, IC4 LDL212PV33R, IC5 LDL212PV33R, IC6 LDL212PV33R, J1 GSB1C41110SSHR, Q10 SSM6K504NU, Q11 SSM6K504NU, Q6 SSM6K504NU, Q7 SSM6K504NU, Q8 SSM6K504NU, Q9 SSM6K504NU, U1 TPSM863252RDXR, U2 ESP32-S3-PICO-1-N8R2

Commit message: Simplify PCB design
Parts:
- removed C1: 22uF, 16V, rcl:C0603
- removed C5, C6, C7: 22uF, rcl:C0603
- removed IC3, IC5: LDL212PV33R, SamacSys_Parts:SON50P200X200X80-7N
- R2: value 200K -> 135K
- R3: value 39K -> 30K
- moved R1 67.0 mm to (-29.2, 0.38), turned to 270 degrees
- moved R3 66.4 mm to (-29.6, 1.91), turned to 180 degrees
- moved R2 65.8 mm to (-29.6, 2.92), turned to 0 degrees
- moved C2 65.2 mm to (-29.6, 3.94), turned to 180 degrees
- moved U1 62.9 mm to (-26.2, 0.89), turned to 90 degrees
- moved C3 61.6 mm to (-26.8, 3.94), turned to 180 degrees
- moved C4 60.2 mm to (-26.8, 5.33), turned to 180 degrees
- moved C20 0.85 mm to (-28.2, -3.17), turned to 0 degrees
- moved C23 0.85 mm to (-28.2, -3.17), turned to 180 degrees
Connections:
- removed net 3V7: C2.1, C3.1, C4.1, C6.1, IC3.4, IC3.6, IC5.4, IC5.6, R2.2, U1.3
- removed net AVCC: C7.1, IC3.2, IC3.3
- net BATT: no longer C1.1
- net DVCC: now also C2.1, C3.1, C4.1, R2.2, U1.3; no longer C5.1, IC5.2, IC5.3
- net GND: no longer C1.2, C5.2, C6.2, C7.2, IC3.1, IC3.7, IC5.1, IC5.7
Routing:
- net DVCC: track 108.3 -> 74.3 mm, vias 7 -> 8
- net 3V7: track 5.08 -> 0.00 mm
- net GND: track 62.9 -> 63.6 mm, vias 29 -> 22
- net BATT: track 10.1 -> 10.6 mm
- removed copper zone on layer 1, net 3V7
- removed copper zone on layer 1, net AVCC

Commit message: v2.1
Parts:
- removed C21, C8, C9: 2.2uF, Customized_components:C0402_STANDARD
- removed IC4, IC6: LDL212PV33R, SamacSys_Parts:SON50P200X200X80-7N
- removed LED2: B38G3RGB-10D0003H2U1930, SamacSys_Parts:B38G3RGB10D0003H2U1930
- removed R40: 1K, Customized_components:R0402_STANDARD
- removed R8: 1.5K, Customized_components:R0402_STANDARD
- removed R9: 820R, Customized_components:R0402_STANDARD
- added C1: 4.7uF, 16V, rcl:C0603
- added C22, C24, C25, C26, C27: 4.7uF, 16V, rcl:C0805
- added C31: 2.2uF, Customized_components:C0402_STANDARD
- added D4: IN4148WT, SamacSys_Parts:SODFL1608X70N
- added IC9: INA231AIYFFR, SamacSys_Parts:BGA12C40P3X4_139X164X62
- added LED1: 150060RS75000, SamacSys_Parts:LEDC1608X80N
- added LED3: SM0605RGB, SamacSys_Parts:SM0605RGB
- added R19: 1K, Customized_components:R0402_STANDARD
- added R20: 1.5K, Customized_components:R0402_STANDARD
- added R21: 820R, Customized_components:R0402_STANDARD
- added R33: 3K, Customized_components:R0402_STANDARD
- added R41: 5mR, rcl:R0805
- added R42, R43: 10K, Customized_components:R0402_STANDARD
- C19: value T523H108M010APE070 -> 4.7uF, 16V; device SamacSys_Parts:CAPPC7260X200N -> rcl:C0805
- C4: value 22uF -> 0.1uF; device rcl:C0603 -> Customized_components:C0402_STANDARD
- R2: value 135K -> 68K
- R3: value 30K -> 15K
- R7: value 820R -> 1.5K
- moved C4 21.4 mm to (-30.4, -15.7), turned to 90 degrees
- moved C20 8.28 mm to (-33.0, -9.91), turned to 90 degrees
- moved C2 6.99 mm to (-33.0, -2.16), turned to 270 degrees
- moved C3 6.93 mm to (-32.9, 0.64), turned to 270 degrees
- moved R5 6.84 mm to (-15.0, 33.9), flipped to the bottom, turned to 270 degrees
- moved C23 6.79 mm to (-27.3, -9.91), flipped to the top, turned to 90 degrees
- moved JP2 5.68 mm to (-38.1, -7.62)
- moved JP3 5.68 mm to (38.1, -7.62)
- moved R2 5.62 mm to (-32.0, -2.16), turned to 90 degrees
- moved R6 5.33 mm to (-13.2, 34.4), flipped to the bottom
- moved R3 4.30 mm to (-31.0, -2.16), turned to 270 degrees
- moved U1 3.70 mm to (-29.8, 1.27), turned to 180 degrees
- moved R4 2.81 mm to (-11.3, 23.7)
- moved C10 2.77 mm to (-11.3, 24.8)
- moved R7 2.36 mm to (-23.2, 22.4)
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Connections:
- net N$45 renamed IO39
- net N$46 renamed IO40
- net N$48 renamed IO41
- net N$49 renamed IO42
- net N$50 renamed IO43
- net N$51 renamed IO44
- removed net GPIO46: U2.52
- removed net IO34_M_CTRL: R40.2, U2.39
- removed net IO35_M_CTRL_FB: IC1.17, R40.1, U2.40
- removed net IO36: U2.41
- removed net IO37: U2.42
- removed net MDVCC: C21.1, IC1.4, IC6.2, IC6.3, R22.2
- removed net N$26: LED2.4, R8.1
- removed net N$5: LED2.1, R7.1
- removed net N$52: U2.51
- removed net N$9: U2.8
- new net BATT_IN: D4.1, IC9.D1, IC9.D2, JP2.2, R41.2
- new net IO34_SCL: IC9.A1, R42.1, U2.39
- new net IO35_SDA: IC9.A2, R43.1, U2.40
- new net IO36_M_CTRL: R19.2, U2.41
- new net IO37_M_CTRL_OUT: IC1.17, R19.1, U2.42
- new net N$27: LED1.2, R33.2
- new net N$29: LED3.2, R21.2
- new net N$37: LED3.3, R20.1
- net 5V: now also D4.2; no longer C8.1, IC4.4, IC4.6
- net BATT: now also C1.1, C22.1, C24.1, C25.1, C26.1, C27.1, IC9.D3, R33.1, R41.1; no longer IC6.4, IC6.6, JP2.2
- net DVCC: now also C31.1, IC1.4, IC9.B1, LED3.1, R22.2, R42.2, R43.2; no longer C9.1, IC4.2, IC4.3, LED2.3
- net GND: now also C1.2, C22.2, C24.2, C25.2, C26.2, C27.2, C31.2, IC9.B3, IC9.C1, IC9.C3, LED1.1; no longer C21.2, C8.2, C9.2, IC4.1, IC4.7, IC6.1, IC6.7
- net IO47_LED_B: now also R21.1; no longer R9.1
- net IO48_LED_R: now also R20.2; no longer R8.2
- net N$4: now also LED3.4, R7.1; no longer LED2.2, R9.2
Routing:
- net IO37_M_CTRL_OUT: track 0.00 -> 39.3 mm, vias 0 -> 2
- net IO35_M_CTRL_FB: track 38.9 -> 0.00 mm, vias 2 -> 0
- net IO35_SDA: track 0.00 -> 37.0 mm, vias 0 -> 2
- net 5V: track 17.6 -> 53.9 mm
- net IO34_SCL: track 0.00 -> 35.4 mm, vias 0 -> 2
- net DVCC: track 74.3 -> 101.8 mm
- net GND: track 63.6 -> 40.5 mm, vias 22 -> 31
- net BATT: track 10.6 -> 25.6 mm, vias 10 -> 9
- net BATT_IN: track 0.00 -> 7.62 mm
- net MDVCC: track 6.54 -> 0.00 mm, vias 1 -> 0
- net IO44: track 0.00 -> 5.50 mm
- net IO42: track 0.00 -> 5.30 mm
- net IO39: track 0.00 -> 5.09 mm
- net IO37: track 4.43 -> 0.00 mm
- net IO36_M_CTRL: track 0.00 -> 4.32 mm
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- added copper zone on layer 16, net BATT
- added copper zone on layer 1, net IO39
- added copper zone on layer 1, net IO40
- added copper zone on layer 1, net IO42
- added copper zone on layer 1, net IO43
- added copper zone on layer 1, net IO44
- added copper zone on layer 1, net IO5
- removed copper zone on layer 1, net IO37
- removed copper zone on layer 1, net MDVCC
Other:
- board size 85 x 81.5 mm -> 85 x 81.6 mm
- board text added: "2025.May.23"
- board text added: "G 40 41 43 G 38 39 G 42 44"
- board text added: "JLCJLCJLCJLC"
- board text added: "Spinon_Test_Platform_2.1"
- board text removed: "2024.Mar.22"
- board text removed: "IO37 IO38 GND GND"
- board text removed: "LDL212PV33R"
- board text removed: "Spinon_2.0"
- board text removed: "TPSM863252"
