File: Electrical/Drone.sch (EAGLE design)
At the start: 76 parts, among them IC1 EFM8BB21F16G-C-QFN20R, IC2 FD6288Q, IC3 LDL212PV33R, IC4 LDL212PV33R, IC5 LDL212PV33R, IC6 LDL212PV33R, J1 GSB1C41110SSHR, Q10 SSM6K504NU, Q11 SSM6K504NU, Q6 SSM6K504NU, Q7 SSM6K504NU, Q8 SSM6K504NU, Q9 SSM6K504NU, U1 TPSM863252RDXR, U2 ESP32-S3-PICO-1-N8R2

Commit message: Simplify PCB design
Parts:
- removed C1: 22uF, 16V, rcl:C-EUC0603
- removed C5, C6, C7: 22uF, rcl:C-EUC0603
- removed IC3, IC5: LDL212PV33R, SamacSys_Parts:LDL212PV33R
- R2: value 200K -> 135K
- R3: value 39K -> 30K
Connections:
- removed net 3V7: C2.1, C3.1, C4.1, C6.1, IC3.EN, IC3.VIN, IC5.EN, IC5.VIN, R2.2, U1.VOUT
- removed net AVCC: C7.1, IC3.ADJ/SENSE, IC3.VOUT
- net BATT: no longer C1.1
- net DVCC: now also C2.1, C3.1, C4.1, R2.2, U1.VOUT; no longer C5.1, IC5.ADJ/SENSE, IC5.VOUT
- net GND: no longer C1.2, C5.2, C6.2, C7.2, IC3.EP, IC3.GND, IC5.EP, IC5.GND
Other:
- moved on the sheet: C20, C23, C4

Commit message: v2.1
Parts:
- removed C21, C8, C9: 2.2uF, Customized_components:C0402_STANDARD
- removed IC4, IC6: LDL212PV33R, SamacSys_Parts:LDL212PV33R
- removed LED2: B38G3RGB-10D0003H2U1930, SamacSys_Parts:B38G3RGB-10D0003H2U1930
- removed R40: 1K, Customized_components:R0402_STANDARD
- removed R8: 1.5K, Customized_components:R0402_STANDARD
- removed R9: 820R, Customized_components:R0402_STANDARD
- added C1: 4.7uF, 16V, rcl:C-EUC0603
- added C22, C24, C25, C26, C27: 4.7uF, 16V, rcl:C-EUC0805
- added C31: 2.2uF, Customized_components:C0402_STANDARD
- added D4: IN4148WT, SamacSys_Parts:IN4148WT
- added IC9: INA231AIYFFR, SamacSys_Parts:INA231AIYFFR
- added LED1: 150060RS75000, SamacSys_Parts:150060RS75000
- added LED3: SM0605RGB, SamacSys_Parts:SM0605RGB
- added R19: 1K, Customized_components:R0402_STANDARD
- added R20: 1.5K, Customized_components:R0402_STANDARD
- added R21: 820R, Customized_components:R0402_STANDARD
- added R33: 3K, Customized_components:R0402_STANDARD
- added R41: 5mR, rcl:R-EU_R0805
- added R42, R43: 10K, Customized_components:R0402_STANDARD
- C19: value T523H108M010APE070 -> 4.7uF, 16V; device SamacSys_Parts:T523H108M010APE070 -> rcl:C-EUC0805
- C4: value 22uF -> 0.1uF; device rcl:C-EUC0603 -> Customized_components:C0402_STANDARD
- R2: value 135K -> 68K
- R3: value 30K -> 15K
- R7: value 820R -> 1.5K
Connections:
- net N$45 renamed IO39
- net N$46 renamed IO40
- net N$48 renamed IO41
- net N$49 renamed IO42
- net N$50 renamed IO43
- net N$51 renamed IO44
- removed net GPIO46: U2.GPIO46
- removed net IO34_M_CTRL: R40.2, U2.GPIO34
- removed net IO35_M_CTRL_FB: IC1.P0.5, R40.1, U2.GPIO35
- removed net IO36: U2.GPIO36
- removed net IO37: U2.GPIO37
- removed net MDVCC: C21.1, IC1.VDD, IC6.ADJ/SENSE, IC6.VOUT, R22.2
- removed net N$26: LED2.K_R, R8.1
- removed net N$5: LED2.K_G, R7.1
- removed net N$52: U2.GPIO45
- removed net N$9: U2.GPIO3
- new net BATT_IN: D4.K, IC9.BUS, IC9.IN-, JP2.2, R41.2
- new net IO34_SCL: IC9.SCL, R42.1, U2.GPIO34
- new net IO35_SDA: IC9.SDA, R43.1, U2.GPIO35
- new net IO36_M_CTRL: R19.2, U2.GPIO36
- new net IO37_M_CTRL_OUT: IC1.P0.5, R19.1, U2.GPIO37
- new net N$27: LED1.A, R33.2
- new net N$29: LED3.CATHODE_BLUE, R21.2
- new net N$37: LED3.CATHODE_RED, R20.1
- net 5V: now also D4.A; no longer C8.1, IC4.EN, IC4.VIN
- net BATT: now also C1.1, C19.1, C22.1, C24.1, C25.1, C26.1, C27.1, IC9.IN+, R33.1, R41.1; no longer C19.+, IC6.EN, IC6.VIN, JP2.2
- net DVCC: now also C31.1, IC1.VDD, IC9.VS, LED3.COMMON_ANODE, R22.2, R42.2, R43.2; no longer C9.1, IC4.ADJ/SENSE, IC4.VOUT, LED2.COM_A
- net GND: now also C1.2, C19.2, C22.2, C24.2, C25.2, C26.2, C27.2, C31.2, IC9.A0, IC9.A1, IC9.GND, LED1.K; no longer C19.-, C21.2, C8.2, C9.2, IC4.EP, IC4.GND, IC6.EP, IC6.GND
- net IO47_LED_B: now also R21.1; no longer R9.1
- net IO48_LED_R: now also R20.2; no longer R8.2
- net N$4: now also LED3.CATHODE_GREEN, R7.1; no longer LED2.K_B, R9.2
Other:
- moved on the sheet: C20, C23, R7
